File: kicad/myFPGA-CLB-slice/carry_chain.kicad_sch (KiCad schematic)
At the start: 11 parts, among them U6 74LS157, U7 74HC86, U8 NC7SB3157P6X

Commit message: fixed kicad names, updated architecure, started CBv
Parts:
- added D? (x4): LED (blue), LED_SMD:LED_0603_1608Metric, symbol Device:LED
- added R? (x4): 330R, Resistor_SMD:R_0805_2012Metric, symbol Device:R
- C10: renamed from C1; Dielectric (none) -> X7R; JLCPCB Part # (none) -> C49678; Part Nr. (none) -> CC0805KRX7R9BB104; Voltage (none) -> 50V
- C11: renamed from C2; Dielectric (none) -> X7R; JLCPCB Part # (none) -> C49678; Part Nr. (none) -> CC0805KRX7R9BB104; Voltage (none) -> 50V
- C12: renamed from C3; Dielectric (none) -> X7R; JLCPCB Part # (none) -> C49678; Part Nr. (none) -> CC0805KRX7R9BB104; Voltage (none) -> 50V
- C13: renamed from C4; Dielectric (none) -> X7R; JLCPCB Part # (none) -> C49678; Part Nr. (none) -> CC0805KRX7R9BB104; Voltage (none) -> 50V
- C14: renamed from C5; Dielectric (none) -> X7R; JLCPCB Part # (none) -> C49678; Part Nr. (none) -> CC0805KRX7R9BB104; Voltage (none) -> 50V
- renumbered U6 to U13, U7 to U8, U8 to U?
Connections:
- net GND: now also D?.1 (K), D?.1 (K), D?.1 (K), D?.1 (K)
- net cout: now also R?.1
- net carry_b: now reaches U8.5, U?.1, U?.4
- net carry_b: now also R?.1
- net carry_c: now reaches U8.2, U?.1, U?.4
- net carry_c: now also R?.1
- net carry_a: now reaches U8.10, U?.1, U?.4
- net carry_a: now also R?.1
- new net: D?.2 (A), R?.2 (x4)

Commit message: kicad -> pcb started
Parts:
- C10, C11, C12, C13, C14: footprint Capacitor_SMD:C_0805_2012Metric -> Capacitor_SMD:C_0603_1608Metric; Dielectric X7R -> (none); JLCPCB Part # C49678 -> (none); Part Nr. CC0805KRX7R9BB104 -> (none); Voltage 50V -> (none)
- R? (x4): footprint Resistor_SMD:R_0805_2012Metric -> Resistor_SMD:R_0603_1608Metric; JLCPCB Part # C17630 -> (none); Part Nr. 0805W8F3300T5E -> (none)

Commit message: kicad: picked JLC parts, fixed routing to match VHDL, started layouting
Parts:
- C10, C11, C12, C13, C14: Dielectric (none) -> X7R; JLCPCB Part # (none) -> C14663; Part Nr. (none) -> CC0603KRX7R9BB104; Voltage (none) -> 50
- R? (x4): JLCPCB Part # (none) -> C23138; Part Nr. (none) -> 0603WAF3300T5E
- U13: JLCPCB Alt # (none) -> C5609 / 74HC157D / SOIC-16-3.9; JLCPCB Part # C5609 -> C6823; Part Nr. 74HC157D -> SN74HC157DR; package (none) -> SOIC-16-3.9
- U8: footprint Package_SO:SOIC-16W_5.3x10.2mm_P1.27mm -> Package_SO:TSSOP-14_4.4x5mm_P0.65mm; JLCPCB Alt # (none) -> C8175 / SN74AHC86DR / SOIC-14-3.9; package (none) -> TSSOP-14-4.4

Commit message: fixed a footprint
Parts:
- U8: package TSSOP-14-4.4 -> (none)
Changed lines of the file:
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@@
       (effects (font (size 1.27 1.27)) hide)
     )
-    (property "package" "TSSOP-14-4.4" (at 166.37 127 0)
+    (property "package" "" (at 166.37 127 0)
       (effects (font (size 1.27 1.27)) hide)
     )
@@
       (effects (font (size 1.27 1.27)) hide)
     )
-    (property "package" "TSSOP-14-4.4" (at 166.37 50.8 0)
+    (property "package" "" (at 166.37 50.8 0)
       (effects (font (size 1.27 1.27)) hide)
     )
@@
       (effects (font (size 1.27 1.27)) hide)
     )
-    (property "package" "TSSOP-14-4.4" (at 166.37 76.2 0)
+    (property "package" "" (at 166.37 76.2 0)
       (effects (font (size 1.27 1.27)) hide)
     )
@@
       (effects (font (size 1.27 1.27)) hide)
     )
-    (property "package" "TSSOP-14-4.4" (at 40.64 129.54 0)
+    (property "package" "" (at 40.64 129.54 0)
       (effects (font (size 1.27 1.27)) hide)
     )
@@
       (effects (font (size 1.27 1.27)) hide)
     )
-    (property "package" "TSSOP-14-4.4" (at 166.37 101.6 0)
-      (effects (font (size 1.27 1.27)) hide)
-    )
+    (property "package" "" (at 166.37 101.6 0)
+      (effects (font (size 1.27 1.27)) hide)
+    )

Commit message: fixed a footprint, changed to 2 Layer stackup
Parts:
- U8: footprint Package_SO:TSSOP-14_4.4x5mm_P0.65mm -> Package_SO:SOIC-14_3.9x8.7mm_P1.27mm; package (none) -> SOIC-14-3.9
Changed lines of the file:
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@@
       (effects (font (size 1.27 1.27)))
     )
-    (property "Footprint" "Package_SO:TSSOP-14_4.4x5mm_P0.65mm" (at 166.37 127 0)
+    (property "Footprint" "Package_SO:SOIC-14_3.9x8.7mm_P1.27mm" (at 166.37 127 0)
       (effects (font (size 1.27 1.27)) hide)
     )
@@
       (effects (font (size 1.27 1.27)) hide)
     )
-    (property "package" "" (at 166.37 127 0)
+    (property "package" "SOIC-14-3.9" (at 166.37 127 0)
       (effects (font (size 1.27 1.27)) hide)
     )
@@
       (effects (font (size 1.27 1.27)))
     )
-    (property "Footprint" "Package_SO:TSSOP-14_4.4x5mm_P0.65mm" (at 166.37 50.8 0)
+    (property "Footprint" "Package_SO:SOIC-14_3.9x8.7mm_P1.27mm" (at 166.37 50.8 0)
       (effects (font (size 1.27 1.27)) hide)
     )
@@
       (effects (font (size 1.27 1.27)) hide)
     )
-    (property "package" "" (at 166.37 50.8 0)
+    (property "package" "SOIC-14-3.9" (at 166.37 50.8 0)
       (effects (font (size 1.27 1.27)) hide)
     )
@@
       (effects (font (size 1.27 1.27)))
     )
-    (property "Footprint" "Package_SO:TSSOP-14_4.4x5mm_P0.65mm" (at 166.37 76.2 0)
+    (property "Footprint" "Package_SO:SOIC-14_3.9x8.7mm_P1.27mm" (at 166.37 76.2 0)
       (effects (font (size 1.27 1.27)) hide)
     )
@@
       (effects (font (size 1.27 1.27)) hide)
     )
-    (property "package" "" (at 166.37 76.2 0)
+    (property "package" "SOIC-14-3.9" (at 166.37 76.2 0)
       (effects (font (size 1.27 1.27)) hide)
     )
@@
       (effects (font (size 1.27 1.27)))
     )
-    (property "Footprint" "Package_SO:TSSOP-14_4.4x5mm_P0.65mm" (at 40.64 129.54 0)
+    (property "Footprint" "Package_SO:SOIC-14_3.9x8.7mm_P1.27mm" (at 40.64 129.54 0)
       (effects (font (size 1.27 1.27)) hide)
     )
@@
       (effects (font (size 1.27 1.27)) hide)
     )
-    (property "package" "" (at 40.64 129.54 0)
+    (property "package" "SOIC-14-3.9" (at 40.64 129.54 0)
       (effects (font (size 1.27 1.27)) hide)
     )
@@
       (effects (font (size 1.27 1.27)))
     )
-    (property "Footprint" "Package_SO:TSSOP-14_4.4x5mm_P0.65mm" (at 166.37 101.6 0)
+    (property "Footprint" "Package_SO:SOIC-14_3.9x8.7mm_P1.27mm" (at 166.37 101.6 0)
       (effects (font (size 1.27 1.27)) hide)
     )
@@
       (effects (font (size 1.27 1.27)) hide)
     )
-    (property "package" "" (at 166.37 101.6 0)
-      (effects (font (size 1.27 1.27)) hide)
-    )
+    (property "package" "SOIC-14-3.9" (at 166.37 101.6 0)
+      (effects (font (size 1.27 1.27)) hide)
+    )

Commit message: more kicad layouts
Parts:
- gave numbers to parts that had none: 12
