File: kicad/myFPGA-CLB-slice/d-latch-register.kicad_sch (KiCad schematic)
At the start: 10 parts, among them U5 74LS175, U8 NC7SB3157P6X

Commit message: fixed kicad names, updated architecure, started CBv
Parts:
- added D? (x4): LED (blue), LED_SMD:LED_0603_1608Metric, symbol Device:LED
- added R? (x4): 330R, Resistor_SMD:R_0805_2012Metric, symbol Device:R
- C?: renamed from C4; Dielectric (none) -> X7R; JLCPCB Part # (none) -> C49678; Part Nr. (none) -> CC0805KRX7R9BB104; Voltage (none) -> 50V
- C?: renamed from C1; Dielectric (none) -> X7R; JLCPCB Part # (none) -> C49678; Part Nr. (none) -> CC0805KRX7R9BB104; Voltage (none) -> 50V
- C?: renamed from C3; Dielectric (none) -> X7R; JLCPCB Part # (none) -> C49678; Part Nr. (none) -> CC0805KRX7R9BB104; Voltage (none) -> 50V
- C?: renamed from C5; Dielectric (none) -> X7R; JLCPCB Part # (none) -> C49678; Part Nr. (none) -> CC0805KRX7R9BB104; Voltage (none) -> 50V
- C?: renamed from C2; Dielectric (none) -> X7R; JLCPCB Part # (none) -> C49678; Part Nr. (none) -> CC0805KRX7R9BB104; Voltage (none) -> 50V
- renumbered U5 to U18, U8 to U?
Connections:
- net Ua is gone; now on net Oa: U18.13 (D3), U?.3
- net Ub is gone; now on net Ob: U18.12 (D2), U?.3
- net Uc is gone; now on net Oc: U18.5 (D1), U?.3
- net Ud is gone; now on net Od: U18.4 (D0), U?.3
- net GND: now also D?.1 (K), D?.1 (K), D?.1 (K), D?.1 (K)
- net Oa: no longer U?.4
- net Ob: no longer U?.4
- net Oc: no longer U?.4
- net Od: no longer U?.4
- net Qd_reg: now reaches U18.2 (Q0), U?.1
- net Qc_reg: now reaches U18.7 (Q1), U?.1
- net Qb_reg: now reaches U18.10 (Q2), U?.1
- net Qa_reg: now reaches U18.15 (Q3), U?.1
- new net: D?.2 (A), R?.2 (x4)
- new net Qa: R?.1, U?.4
- new net Qb: R?.1, U?.4
- new net Qc: R?.1, U?.4
- new net Qd: R?.1, U?.4

Commit message: kicad -> pcb started
Parts:
- C? (x5): footprint Capacitor_SMD:C_0805_2012Metric -> Capacitor_SMD:C_0603_1608Metric; Dielectric X7R -> (none); JLCPCB Part # C49678 -> (none); Part Nr. CC0805KRX7R9BB104 -> (none); Voltage 50V -> (none)
- R? (x4): footprint Resistor_SMD:R_0805_2012Metric -> Resistor_SMD:R_0603_1608Metric; JLCPCB Part # C17630 -> (none); Part Nr. 0805W8F3300T5E -> (none)

Commit message: kicad: picked JLC parts, fixed routing to match VHDL, started layouting
Parts:
- C? (x5): Dielectric (none) -> X7R; JLCPCB Part # (none) -> C14663; Part Nr. (none) -> CC0603KRX7R9BB104; Voltage (none) -> 50
- R? (x4): JLCPCB Part # (none) -> C23138; Part Nr. (none) -> 0603WAF3300T5E
- U18: footprint Package_SO:SOIC-16W_5.3x10.2mm_P1.27mm -> Package_SO:SOIC-16_3.9x9.9mm_P1.27mm; JLCPCB Alt # (none) -> C546669 / 74HC175PW / TSSOP-16; JLCPCB Part # C7745 -> C8180; Part Nr. SN74LS175DR -> CD74AC175M96; package (none) -> SOIC-16-3.9

Commit message: progress in pcb of CLB
Connections:
- net +3V3: no longer U18.1 (~{Mr})
- new net aresetn: U18.1 (~{Mr})
Changed lines of the file:
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@@
+    (stroke (width 0) (type default))
+  )
+  (wire (pts (xy 101.6 146.05) (xy 120.65 146.05))
     (stroke (width 0) (type default))
   )
@@
   )
   (hierarchical_label "Oa" (shape input) (at 101.6 138.43 180) (fields_autoplaced)
+    (effects (font (size 1.27 1.27)) (justify right))
+  )
+  (hierarchical_label "aresetn" (shape input) (at 101.6 146.05 180) (fields_autoplaced)
     (effects (font (size 1.27 1.27)) (justify right))
   )
@@
         )
       )
-    )
-  )
-  (symbol (lib_id "power:+3V3") (at 120.65 146.05 90) (unit 1)
-    (in_bom yes) (on_board yes) (dnp no) (fields_autoplaced)
-    (property "Reference" "#PWR?" (at 124.46 146.05 0)
-      (effects (font (size 1.27 1.27)) hide)
-    )
-    (property "Value" "+3V3" (at 116.84 146.05 90)
-      (effects (font (size 1.27 1.27)) (justify left))
-    )
-    (property "Footprint" "" (at 120.65 146.05 0)
-      (effects (font (size 1.27 1.27)) hide)
-    )
-    (property "Datasheet" "" (at 120.65 146.05 0)
-      (effects (font (size 1.27 1.27)) hide)
-    )
-    (pin "1")
-    (instances
-      (project "myFPGA-CLB-slice"
-        (path "/2d29d97f-956a-4594-9321-3d88807a498d/2ae8c962-eb3a-4bc0-879b-9a9a0cb7ca8b"
-          (reference "#PWR?") (unit 1)
-        )
-        (path "/2d29d97f-956a-4594-9321-3d88807a498d/8bde6bd0-53b6-4d4d-9e74-d6add268472f"
-          (reference "#PWR055") (unit 1)
-        )
-      )

Commit message: more kicad layouts
Parts:
- gave numbers to parts that had none: 17
