File: kicad/myFPGA-CLB-slice/lut4.kicad_sch (KiCad schematic)
At the start: 10 parts, among them U1 74AHCT595, U3 74LS151, U4 74LS151, U8 NC7SB3157P6X

Commit message: fixed kicad names, updated architecure, started CBv
Parts:
- C?: renamed from C5; Dielectric (none) -> X7R; JLCPCB Part # (none) -> C49678; Part Nr. (none) -> CC0805KRX7R9BB104; Voltage (none) -> 50V
- C?: renamed from C2; Dielectric (none) -> X7R; JLCPCB Part # (none) -> C49678; Part Nr. (none) -> CC0805KRX7R9BB104; Voltage (none) -> 50V
- C?: renamed from C1; Dielectric (none) -> X7R; JLCPCB Part # (none) -> C49678; Part Nr. (none) -> CC0805KRX7R9BB104; Voltage (none) -> 50V
- C?: renamed from C4; Dielectric (none) -> X7R; JLCPCB Part # (none) -> C49678; Part Nr. (none) -> CC0805KRX7R9BB104; Voltage (none) -> 50V
- C?: renamed from C3; Dielectric (none) -> X7R; JLCPCB Part # (none) -> C49678; Part Nr. (none) -> CC0805KRX7R9BB104; Voltage (none) -> 50V
- renumbered U3 to U5, U4 to U6, U8 to U?, U1 to U?

Commit message: kicad -> pcb started
Parts:
- C? (x5): footprint Capacitor_SMD:C_0805_2012Metric -> Capacitor_SMD:C_0603_1608Metric; Dielectric X7R -> (none); JLCPCB Part # C49678 -> (none); Part Nr. CC0805KRX7R9BB104 -> (none); Voltage 50V -> (none)

Commit message: kicad: picked JLC parts, fixed routing to match VHDL, started layouting
Parts:
- C? (x5): Dielectric (none) -> X7R; JLCPCB Part # (none) -> C14663; Part Nr. (none) -> CC0603KRX7R9BB104; Voltage (none) -> 50
- U5, U6: footprint Package_SO:SOIC-16W_5.3x10.2mm_P1.27mm -> Package_SO:TSSOP-16_4.4x5mm_P0.65mm; JLCPCB Alt # (none) -> C6822 / SN74HC151DR / SOIC-16-3.9; JLCPCB Part # C6822 -> C152523; Part Nr. SN74HC151DR -> MC74HC151ADTR2G; package (none) -> TSSOP-16-4.4
- U? (x2): JLCPCB Alt # (none) -> C431479 / 74HC595D / SOIC-16-3.9; package (none) -> SOIC-16-3.9
Connections:
- net +3V3: no longer C?.1, C?.1, C?.1, C?.1, U5.16 (VCC), U6.16 (VCC), U?.16 (VCC), U?.16 (VCC)
- new net +3.3VP: C?.1, C?.1, C?.1, C?.1, U6.16 (VCC), U?.16 (VCC), U?.16 (VCC)

Commit message: restart PCB layout
Connections:
- net +3.3VP: now also U5.16 (VCC)
- net REG renamed LATCH
Changed lines of the file:
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@@
     (effects (font (size 1.27 1.27)) (justify right))
   )
-  (hierarchical_label "REG" (shape input) (at 78.74 58.42 180) (fields_autoplaced)
+  (hierarchical_label "LATCH" (shape input) (at 78.74 58.42 180) (fields_autoplaced)
     (effects (font (size 1.27 1.27)) (justify right))
   )
@@
         )
       )
+    )
+  )
+  (symbol (lib_id "power:+3.3VP") (at 132.08 38.1 0) (unit 1)
+    (in_bom yes) (on_board yes) (dnp no)
+    (property "Reference" "#PWR013" (at 135.89 39.37 0)
+      (effects (font (size 1.27 1.27)) hide)
+    )
+    (property "Value" "+3.3VP" (at 132.08 33.02 0)
+      (effects (font (size 1.27 1.27)))
+    )
+    (property "Footprint" "" (at 132.08 38.1 0)
+      (effects (font (size 1.27 1.27)) hide)
+    )
+    (property "Datasheet" "" (at 132.08 38.1 0)
+      (effects (font (size 1.27 1.27)) hide)
+    )
+    (pin "1")
+    (instances
+      (project "myFPGA-CLB-slice"
+        (path "/2d29d97f-956a-4594-9321-3d88807a498d"
+          (reference "#PWR013") (unit 1)
+        )
+        (path "/2d29d97f-956a-4594-9321-3d88807a498d/2ae8c962-eb3a-4bc0-879b-9a9a0cb7ca8b"
+          (reference "#PWR06") (unit 1)
+        )
+        (path "/2d29d97f-956a-4594-9321-3d88807a498d/c0683758-8f95-4956-98b3-1cadd07503a7"
+          (reference "#PWR0140") (unit 1)
+        )
+        (path "/2d29d97f-956a-4594-9321-3d88807a498d/8d6c6a11-91f4-4cda-a0a3-b01338b326ab"
+          (reference "#PWR0141") (unit 1)
+        )
+        (path "/2d29d97f-956a-4594-9321-3d88807a498d/f8f5aa5a-daee-44c0-974a-67be9fa42cb8"
+          (reference "#PWR0142") (unit 1)
+        )
+      )

Commit message: gitignore fix
Connections:
- net +3.3VP: now also U?.10 (~{SRCLR}), U?.10 (~{SRCLR})
- net GND: no longer U?.10 (~{SRCLR}), U?.10 (~{SRCLR})
Changed lines of the file:
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@@
   (junction (at 49.53 184.15) (diameter 0) (color 0 0 0 0)
   )
-  (junction (at 87.63 121.92) (diameter 0) (color 0 0 0 0)
-  )
   (junction (at 83.82 50.8) (diameter 0) (color 0 0 0 0)
   )
-  (junction (at 87.63 60.96) (diameter 0) (color 0 0 0 0)
-  )
   (junction (at 85.09 58.42) (diameter 0) (color 0 0 0 0)
   )
@@
   )
   (junction (at 116.84 134.62) (diameter 0) (color 0 0 0 0)
+  )
+  (junction (at 82.55 53.34) (diameter 0) (color 0 0 0 0)
   )
   (junction (at 43.18 184.15) (diameter 0) (color 0 0 0 0)
@@
     (stroke (width 0) (type default))
   )
-  (wire (pts (xy 88.9 114.3) (xy 87.63 114.3))
+  (wire (pts (xy 82.55 114.3) (xy 88.9 114.3))
     (stroke (width 0) (type default))
   )
@@
     (stroke (width 0) (type default))
   )
-  (wire (pts (xy 87.63 53.34) (xy 87.63 60.96))
-    (stroke (width 0) (type default))
-  )
   (wire (pts (xy 87.63 121.92) (xy 87.63 134.62))
     (stroke (width 0) (type default))
@@
     (stroke (width 0) (type default))
   )
+  (wire (pts (xy 82.55 40.64) (xy 82.55 53.34))
+    (stroke (width 0) (type default))
+  )
   (wire (pts (xy 30.48 184.15) (xy 36.83 184.15))
     (stroke (width 0) (type default))
@@
     (stroke (width 0) (type default))
   )
-  (wire (pts (xy 88.9 53.34) (xy 87.63 53.34))
+  (wire (pts (xy 82.55 53.34) (xy 88.9 53.34))
     (stroke (width 0) (type default))
   )
@@
     (stroke (width 0) (type default))
   )
+  (wire (pts (xy 82.55 53.34) (xy 82.55 114.3))
+    (stroke (width 0) (type default))
+  )
   (wire (pts (xy 115.57 71.12) (xy 115.57 132.08))
     (stroke (width 0) (type default))
@@
   )
   (wire (pts (xy 161.29 55.88) (xy 161.29 157.48))
-    (stroke (width 0) (type default))
-  )
-  (wire (pts (xy 87.63 114.3) (xy 87.63 121.92))
     (stroke (width 0) (type default))
   )
@@
         )
       )
+    )
+  )
+  (symbol (lib_id "power:+3.3VP") (at 82.55 40.64 0) (unit 1)
+    (in_bom yes) (on_board yes) (dnp no)
+    (property "Reference" "#PWR013" (at 86.36 41.91 0)
+      (effects (font (size 1.27 1.27)) hide)
+    )
+    (property "Value" "+3.3VP" (at 82.55 35.56 0)
+      (effects (font (size 1.27 1.27)))
+    )
+    (property "Footprint" "" (at 82.55 40.64 0)
+      (effects (font (size 1.27 1.27)) hide)
+    )
+    (property "Datasheet" "" (at 82.55 40.64 0)
+      (effects (font (size 1.27 1.27)) hide)
+    )
+    (pin "1")
+    (instances
+      (project "myFPGA-CLB-slice"
+        (path "/2d29d97f-956a-4594-9321-3d88807a498d"
+          (reference "#PWR013") (unit 1)
+        )
+        (path "/2d29d97f-956a-4594-9321-3d88807a498d/2ae8c962-eb3a-4bc0-879b-9a9a0cb7ca8b"
+          (reference "#PWR0148") (unit 1)
+        )
+        (path "/2d29d97f-956a-4594-9321-3d88807a498d/c0683758-8f95-4956-98b3-1cadd07503a7"
+          (reference "#PWR0149") (unit 1)
+        )
+        (path "/2d29d97f-956a-4594-9321-3d88807a498d/8d6c6a11-91f4-4cda-a0a3-b01338b326ab"
+          (reference "#PWR0150") (unit 1)
+        )
+        (path "/2d29d97f-956a-4594-9321-3d88807a498d/f8f5aa5a-daee-44c0-974a-67be9fa42cb8"
+          (reference "#PWR0151") (unit 1)
+        )
+      )

Commit message: more kicad layouts
Parts:
- gave numbers to parts that had none: 8
Changed lines of the file:
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@@
   (symbol (lib_id "Device:C") (at 49.53 180.34 0) (unit 1)
     (in_bom yes) (on_board yes) (dnp no)
-    (property "Reference" "C?" (at 48.26 170.18 0)
+    (property "Reference" "C9" (at 48.26 170.18 0)
       (effects (font (size 1.27 1.27)) (justify left))
     )
@@
     (instances
       (project "myFPGA-CLB-slice"
-        (path "/2d29d97f-956a-4594-9321-3d88807a498d/4edb728f-4165-4dad-bea7-d5caa521ea2d"
-          (reference "C?") (unit 1)
-        )
         (path "/2d29d97f-956a-4594-9321-3d88807a498d/2ae8c962-eb3a-4bc0-879b-9a9a0cb7ca8b"
           (reference "C9") (unit 1)
@@
   (symbol (lib_id "power:+3.3VP") (at 132.08 99.06 0) (unit 1)
     (in_bom yes) (on_board yes) (dnp no)
-    (property "Reference" "#PWR013" (at 135.89 100.33 0)
+    (property "Reference" "#PWR028" (at 135.89 100.33 0)
       (effects (font (size 1.27 1.27)) hide)
     )
@@
     (instances
       (project "myFPGA-CLB-slice"
-        (path "/2d29d97f-956a-4594-9321-3d88807a498d"
-          (reference "#PWR013") (unit 1)
-        )
         (path "/2d29d97f-956a-4594-9321-3d88807a498d/2ae8c962-eb3a-4bc0-879b-9a9a0cb7ca8b"
           (reference "#PWR028") (unit 1)
@@
   (symbol (lib_id "power:+3.3VP") (at 99.06 101.6 0) (unit 1)
     (in_bom yes) (on_board yes) (dnp no)
-    (property "Reference" "#PWR013" (at 102.87 102.87 0)
+    (property "Reference" "#PWR066" (at 102.87 102.87 0)
       (effects (font (size 1.27 1.27)) hide)
     )
@@
     (instances
       (project "myFPGA-CLB-slice"
-        (path "/2d29d97f-956a-4594-9321-3d88807a498d"
-          (reference "#PWR013") (unit 1)
-        )
         (path "/2d29d97f-956a-4594-9321-3d88807a498d/2ae8c962-eb3a-4bc0-879b-9a9a0cb7ca8b"
           (reference "#PWR066") (unit 1)
@@
   (symbol (lib_id "Analog_Switch:NC7SB3157P6X") (at 161.29 45.72 0) (mirror y) (unit 1)
     (in_bom yes) (on_board yes) (dnp no)
-    (property "Reference" "U?" (at 162.56 39.37 0)
+    (property "Reference" "U7" (at 162.56 39.37 0)
       (effects (font (size 1.27 1.27)))
     )
@@
     (instances
       (project "myFPGA-CLB-slice"
-        (path "/2d29d97f-956a-4594-9321-3d88807a498d"
-          (reference "U?") (unit 1)
-        )
-        (path "/2d29d97f-956a-4594-9321-3d88807a498d/4edb728f-4165-4dad-bea7-d5caa521ea2d"
-          (reference "U?") (unit 1)
-        )
         (path "/2d29d97f-956a-4594-9321-3d88807a498d/2ae8c962-eb3a-4bc0-879b-9a9a0cb7ca8b"
           (reference "U7") (unit 1)
@@
   (symbol (lib_id "Analog_Switch:NC7SB3157P6X") (at 153.67 182.88 90) (mirror x) (unit 2)
     (in_bom yes) (on_board yes) (dnp no)
-    (property "Reference" "U?" (at 163.83 177.8 90)
+    (property "Reference" "U7" (at 163.83 177.8 90)
       (effects (font (size 1.27 1.27)) (justify left))
     )
@@
     (instances
       (project "myFPGA-CLB-slice"
-        (path "/2d29d97f-956a-4594-9321-3d88807a498d"
-          (reference "U?") (unit 2)
-        )
-        (path "/2d29d97f-956a-4594-9321-3d88807a498d/4edb728f-4165-4dad-bea7-d5caa521ea2d"
-          (reference "U?") (unit 2)
-        )
         (path "/2d29d97f-956a-4594-9321-3d88807a498d/2ae8c962-eb3a-4bc0-879b-9a9a0cb7ca8b"
           (reference "U7") (unit 2)
@@
   (symbol (lib_id "power:+3.3VP") (at 55.88 173.99 0) (unit 1)
     (in_bom yes) (on_board yes) (dnp no)
-    (property "Reference" "#PWR013" (at 59.69 175.26 0)
+    (property "Reference" "#PWR098" (at 59.69 175.26 0)
       (effects (font (size 1.27 1.27)) hide)
     )
@@
     (instances
       (project "myFPGA-CLB-slice"
-        (path "/2d29d97f-956a-4594-9321-3d88807a498d"
-          (reference "#PWR013") (unit 1)
-        )
         (path "/2d29d97f-956a-4594-9321-3d88807a498d/2ae8c962-eb3a-4bc0-879b-9a9a0cb7ca8b"
           (reference "#PWR098") (unit 1)
@@
   (symbol (lib_id "power:+3.3VP") (at 82.55 40.64 0) (unit 1)
     (in_bom yes) (on_board yes) (dnp no)
-    (property "Reference" "#PWR013" (at 86.36 41.91 0)
+    (property "Reference" "#PWR0148" (at 86.36 41.91 0)
       (effects (font (size 1.27 1.27)) hide)
     )
@@
     (instances
       (project "myFPGA-CLB-slice"
-        (path "/2d29d97f-956a-4594-9321-3d88807a498d"
-          (reference "#PWR013") (unit 1)
-        )
         (path "/2d29d97f-956a-4594-9321-3d88807a498d/2ae8c962-eb3a-4bc0-879b-9a9a0cb7ca8b"
           (reference "#PWR0148") (unit 1)
@@
   (symbol (lib_id "power:+3.3VP") (at 132.08 38.1 0) (unit 1)
     (in_bom yes) (on_board yes) (dnp no)
-    (property "Reference" "#PWR013" (at 135.89 39.37 0)
+    (property "Reference" "#PWR06" (at 135.89 39.37 0)
       (effects (font (size 1.27 1.27)) hide)
     )
@@
     (instances
       (project "myFPGA-CLB-slice"
-        (path "/2d29d97f-956a-4594-9321-3d88807a498d"
-          (reference "#PWR013") (unit 1)
-        )
         (path "/2d29d97f-956a-4594-9321-3d88807a498d/2ae8c962-eb3a-4bc0-879b-9a9a0cb7ca8b"
           (reference "#PWR06") (unit 1)
@@
   (symbol (lib_id "power:+3.3VP") (at 99.06 40.64 0) (unit 1)
     (in_bom yes) (on_board yes) (dnp no)
-    (property "Reference" "#PWR013" (at 102.87 41.91 0)
+    (property "Reference" "#PWR082" (at 102.87 41.91 0)
       (effects (font (size 1.27 1.27)) hide)
     )
@@
     (instances
       (project "myFPGA-CLB-slice"
-        (path "/2d29d97f-956a-4594-9321-3d88807a498d"
-          (reference "#PWR013") (unit 1)
-        )
         (path "/2d29d97f-956a-4594-9321-3d88807a498d/2ae8c962-eb3a-4bc0-879b-9a9a0cb7ca8b"
           (reference "#PWR082") (unit 1)
@@
   (symbol (lib_id "power:GND") (at 55.88 186.69 0) (unit 1)
     (in_bom yes) (on_board yes) (dnp no) (fields_autoplaced)
-    (property "Reference" "#PWR?" (at 55.88 193.04 0)
+    (property "Reference" "#PWR025" (at 55.88 193.04 0)
       (effects (font (size 1.27 1.27)) hide)
     )
@@
     (instances
       (project "myFPGA-CLB-slice"
-        (path "/2d29d97f-956a-4594-9321-3d88807a498d/4edb728f-4165-4dad-bea7-d5caa521ea2d"
-          (reference "#PWR?") (unit 1)
-        )
         (path "/2d29d97f-956a-4594-9321-3d88807a498d/2ae8c962-eb3a-4bc0-879b-9a9a0cb7ca8b"
           (reference "#PWR025") (unit 1)
@@
   (symbol (lib_id "Device:C") (at 30.48 180.34 0) (unit 1)
     (in_bom yes) (on_board yes) (dnp no)
-    (property "Reference" "C?" (at 29.21 170.18 0)
+    (property "Reference" "C6" (at 29.21 170.18 0)
       (effects (font (size 1.27 1.27)) (justify left))
     )
@@
     (instances
       (project "myFPGA-CLB-slice"
-        (path "/2d29d97f-956a-4594-9321-3d88807a498d/4edb728f-4165-4dad-bea7-d5caa521ea2d"
-          (reference "C?") (unit 1)
-        )
         (path "/2d29d97f-956a-4594-9321-3d88807a498d/2ae8c962-eb3a-4bc0-879b-9a9a0cb7ca8b"
           (reference "C6") (unit 1)
@@
   (symbol (lib_id "Device:C") (at 24.13 180.34 0) (unit 1)
     (in_bom yes) (on_board yes) (dnp no)
-    (property "Reference" "C?" (at 17.78 180.34 0)
+    (property "Reference" "C5" (at 17.78 180.34 0)
       (effects (font (size 1.27 1.27)) (justify left))
     )
@@
     (instances
       (project "myFPGA-CLB-slice"
-        (path "/2d29d97f-956a-4594-9321-3d88807a498d/4edb728f-4165-4dad-bea7-d5caa521ea2d"
-          (reference "C?") (unit 1)
-        )
         (path "/2d29d97f-956a-4594-9321-3d88807a498d/2ae8c962-eb3a-4bc0-879b-9a9a0cb7ca8b"
           (reference "C5") (unit 1)
@@
   (symbol (lib_id "Device:C") (at 43.18 180.34 0) (unit 1)
     (in_bom yes) (on_board yes) (dnp no)
-    (property "Reference" "C?" (at 41.91 170.18 0)
+    (property "Reference" "C8" (at 41.91 170.18 0)
       (effects (font (size 1.27 1.27)) (justify left))
     )
@@
     (instances
       (project "myFPGA-CLB-slice"
-        (path "/2d29d97f-956a-4594-9321-3d88807a498d/4edb728f-4165-4dad-bea7-d5caa521ea2d"
-          (reference "C?") (unit 1)
-        )
         (path "/2d29d97f-956a-4594-9321-3d88807a498d/2ae8c962-eb3a-4bc0-879b-9a9a0cb7ca8b"
           (reference "C8") (unit 1)
@@
   (symbol (lib_id "Device:C") (at 36.83 180.34 0) (unit 1)
     (in_bom yes) (on_board yes) (dnp no)
-    (property "Reference" "C?" (at 35.56 170.18 0)
+    (property "Reference" "C7" (at 35.56 170.18 0)
       (effects (font (size 1.27 1.27)) (justify left))
     )
@@
     (instances
       (project "myFPGA-CLB-slice"
-        (path "/2d29d97f-956a-4594-9321-3d88807a498d/4edb728f-4165-4dad-bea7-d5caa521ea2d"
-          (reference "C?") (unit 1)
-        )
         (path "/2d29d97f-956a-4594-9321-3d88807a498d/2ae8c962-eb3a-4bc0-879b-9a9a0cb7ca8b"
           (reference "C7") (unit 1)
@@
   (symbol (lib_id "74xx:74AHCT595") (at 99.06 116.84 0) (unit 1)
     (in_bom yes) (on_board yes) (dnp no) (fields_autoplaced)
-    (property "Reference" "U?" (at 101.2541 99.06 0)
+    (property "Reference" "U4" (at 101.2541 99.06 0)
       (effects (font (size 1.27 1.27)) (justify left))
     )
@@
     (instances
       (project "myFPGA-CLB-slice"
-        (path "/2d29d97f-956a-4594-9321-3d88807a498d"
-          (reference "U?") (unit 1)
-        )
         (path "/2d29d97f-956a-4594-9321-3d88807a498d/2ae8c962-eb3a-4bc0-879b-9a9a0cb7ca8b"
           (reference "U4") (unit 1)
@@
   (symbol (lib_id "74xx:74AHCT595") (at 99.06 55.88 0) (unit 1)
     (in_bom yes) (on_board yes) (dnp no) (fields_autoplaced)
-    (property "Reference" "U?" (at 101.2541 38.1 0)
+    (property "Reference" "U3" (at 101.2541 38.1 0)
       (effects (font (size 1.27 1.27)) (justify left))
     )
@@
     (instances
       (project "myFPGA-CLB-slice"
-        (path "/2d29d97f-956a-4594-9321-3d88807a498d"
-          (reference "U?") (unit 1)
-        )
         (path "/2d29d97f-956a-4594-9321-3d88807a498d/2ae8c962-eb3a-4bc0-879b-9a9a0cb7ca8b"
           (reference "U3") (unit 1)
