File: kicad/myFPGA-CBv/myFPGA-CBv.kicad_sch (KiCad schematic)
At the start: 52 parts, among them J1 Conn_01x04, J10 Conn_01x04, J2 Conn_01x04, J3 Conn_01x04, J4 Conn_01x04, J5 Conn_01x02, J6 Conn_01x02, J6 Conn_01x04, J7 Conn_01x04, J9 Conn_01x04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

Commit message: more kicad layouts 2.
Changed lines of the file:
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@@
     (effects (font (size 1.27 1.27)) (justify left bottom))
   )
-  (label "s_0" (at 140.97 149.86 0) (fields_autoplaced)
+  (label "s_0" (at 132.08 149.86 0) (fields_autoplaced)
     (effects (font (size 1.27 1.27)) (justify left bottom))
   )
-  (label "s_3" (at 140.97 96.52 0) (fields_autoplaced)
+  (label "s_3" (at 132.08 96.52 0) (fields_autoplaced)
     (effects (font (size 1.27 1.27)) (justify left bottom))
   )
-  (label "s_1" (at 140.97 132.08 0) (fields_autoplaced)
+  (label "s_1" (at 134.62 132.08 0) (fields_autoplaced)
     (effects (font (size 1.27 1.27)) (justify left bottom))
   )
-  (label "s_2" (at 140.97 114.3 0) (fields_autoplaced)
+  (label "s_2" (at 134.62 114.3 0) (fields_autoplaced)
     (effects (font (size 1.27 1.27)) (justify left bottom))
   )
