File: kicad/myFPGA-SW-box/myFPGA-SW-box.kicad_pcb (KiCad board)
At the start: 4 copper layers, 90 x 80 mm, 118 parts, among them J1 Conn_01x04, J10 Conn_01x02, J11 Conn_01x02, J12 Conn_01x02, J2 Conn_01x04, J3 Conn_01x04, J4 Conn_01x04, J5 Conn_01x04, J6 Conn_01x04, J7 Conn_01x04, J8 Conn_01x02, J9 Conn_01x04, U1 74HC595, U10 NC7SB3157P6X, U11 NC7SB3157P6X, U12 NC7SB3157P6X, U13 NC7SB3157P6X, U14 NC7SB3157P6X, U15 NC7SB3157P6X, U16 NC7SB3157P6X, U17 NC7SB3157P6X, U18 NC7SB3157P6X, U19 NC7SB3157P6X, U2 74HC595, U20 NC7SB3157P6X, U21 NC7SB3157P6X, U22 NC7SB3157P6X, U23 NC7SB3157P6X, U24 NC7SB3157P6X, U25 NC7SB3157P6X, U26 NC7SB3157P6X, U27 NC7SB3157P6X, U28 NC7SB3157P6X, U29 NC7SB3157P6X, U3 74HC595, U30 NC7SB3157P6X, U31 NC7SB3157P6X, U32 NC7SB3157P6X, U33 NC7SB3157P6X, U34 NC7SB3157P6X, U35 NC7SB3157P6X, U36 NC7SB3157P6X, U4 74HC595, U5 NC7SB3157P6X, U6 NC7SB3157P6X, U7 NC7SB3157P6X, U8 NC7SB3157P6X, U9 NC7SB3157P6X

Commit message: found more bugs
Parts:
- moved J2 1.00 mm to (105.0, 55.6)
- moved J3 1.00 mm to (105.0, 75.6)
- moved J8 1.00 mm to (105.0, 63.5)
Routing:
- net GND: track 205.6 -> 218.4 mm, vias 40 -> 41
- net +3.3VP: track 86.5 -> 95.9 mm, vias 39 -> 40
- net SCLK: track 230.6 -> 229.6 mm
- net MISO: track 16.5 -> 15.5 mm
- net LATCH: track 234.2 -> 233.2 mm
- net /west_2: track 11.4 -> 10.4 mm
- net /west_1: track 13.5 -> 12.5 mm
- net /west_0: track 16.7 -> 15.7 mm
- net /prio_west_1: track 11.2 -> 10.2 mm
- net /prio_west_0: track 10.1 -> 9.15 mm
- net /west_3: track 10.4 -> 9.37 mm
Other:
- outline, holes or cut-outs redrawn
- board text added: "4"
- board text added: "5"
- board text added: "C"
- board text added: "DI"
- board text added: "DO"
- board text added: "L"
